File: doc/pcb/lightring2/lightring.kicad_pcb (KiCad board)
At the start: 2 copper layers, 44 x 44 mm, 113 parts, among them SW1 SW_SPST, SW2 SW_SPST, U1 STM32G070RBT, Y1 Crystal

Commit message: v2 base board
Parts:
- moved R15 53.9 mm to (147.6, 59.1)
- moved R22 53.9 mm to (151.6, 59.0)
- moved R16 53.9 mm to (139.5, 66.9)
- moved R17 53.9 mm to (143.5, 64.2)
- moved R18 53.9 mm to (151.6, 56.5)
- moved R21 53.9 mm to (147.6, 61.6)
- moved R23 53.9 mm to (143.5, 66.7)
- moved R24 53.9 mm to (147.5, 64.1)
- moved R26 53.9 mm to (143.5, 69.2)
- moved R27 53.9 mm to (151.6, 61.5)
- moved R20 53.9 mm to (143.5, 61.7)
- moved R28 29.9 mm to (195.8, 84.2)
- moved R25 29.9 mm to (195.8, 81.7)
- moved R14 29.9 mm to (195.9, 76.5)
- moved R19 29.9 mm to (195.9, 79.1)
Routing:
- net Net-(D24-Pad2): track 33.0 -> 0.00 mm, vias 2 -> 0
- net Net-(D21-Pad2): track 32.7 -> 0.00 mm, vias 2 -> 0
- net Net-(D23-Pad2): track 32.2 -> 0.00 mm, vias 2 -> 0
- net Net-(D22-Pad2): track 31.2 -> 0.00 mm, vias 2 -> 0
- net Net-(D20-Pad2): track 30.7 -> 0.00 mm, vias 2 -> 0
- net Net-(D17-Pad2): track 29.5 -> 0.00 mm
- net Net-(D18-Pad2): track 29.5 -> 0.00 mm, vias 2 -> 0
- net Net-(D19-Pad2): track 29.4 -> 0.00 mm, vias 2 -> 0
- net VCC: track 27.8 -> 0.00 mm, vias 1 -> 0
- net Net-(D10-Pad2): track 18.2 -> 0.00 mm, vias 1 -> 0
- net XTAL1: track 9.76 -> 0.00 mm
- net XTAL2: track 6.25 -> 0.00 mm
