File: doc/pcb/lightring1/lightring.kicad_pcb (KiCad board)
At the start: 2 copper layers, 44 x 44 mm, 114 parts, among them J1 Conn_01x05_Female, J2 USB_B_Micro, J3 plate, SW2 SW_SPST, U1 STM32G070RBT, U2 MCP73831-2-OT, U3 AT42QT1012-T, U4 LDK130-33_SOT23_SOT353, Y1 Crystal

Commit message: v0.3 PCB
Parts:
- added C3: 104, Capacitor_SMD:C_0603_1608Metric, B.Cu at (169.6, 65.8)
- added R50: 100k, Resistor_SMD:R_0603_1608Metric, B.Cu at (166.6, 65.7)
- added R51: 100k, Resistor_SMD:R_0603_1608Metric, B.Cu at (166.6, 67.2)
- BT1: footprint Resistor_SMD:R_1206_3216Metric -> Resistor_SMD:R_1210_3225Metric
- moved BT1 0.06 mm to (164.6, 61.0)
Connections:
- U1 pad 17: M20 -> STATE
- U1 pad 41: Net-(U1-Pad41) -> M20
Routing:
- net M20: track 21.8 -> 77.0 mm, vias 2 -> 4
- net STATE: track 0.00 -> 36.6 mm, vias 0 -> 2
- net Net-(J3-Pad1): track 9.36 -> 14.0 mm
- net Net-(U1-Pad41): track 2.68 -> 0.00 mm
- net Net-(J1-Pad1): track 19.7 -> 22.2 mm
- net GND: track 371.2 -> 373.7 mm
- net VCC: track 50.4 -> 48.5 mm
- net M1: track 15.4 -> 16.9 mm
- net M29: track 13.2 -> 14.0 mm
- net +3V3: track 49.2 -> 49.1 mm, vias 1 -> 3
Other:
- board text added: "+"
- board text added: "-"
