File: doc/pcb/lightring1/lightring.sch (KiCad schematic (older format))
At the start: 101 parts, among them J1 Conn_01x05_Female, SW1 SW_SPST, SW2 SW_SPST, U1 STM32G070RBT, Y1 Crystal

Commit message: v0.2 board
Parts:
- removed C3: 105, lightring:LC_CAP, symbol Device:C
- removed SW1: SW_SPST, Button_Switch_SMD:Panasonic_EVQPUJ_EVQPUA, symbol Switch:SW_SPST
- added C10: 100nF, Capacitor_SMD:C_0603_1608Metric, symbol Device:C
- added C11: 2.2n, Capacitor_SMD:C_0603_1608Metric, symbol Device:C
- added C12: 105, Capacitor_SMD:C_0603_1608Metric, symbol Device:C
- added C9: 475, Capacitor_SMD:C_0603_1608Metric, symbol Device:C
- added D44: LED, Diode_SMD:D_0603_1608Metric, symbol Device:LED
- added J2: USB_B_Micro, Connector_USB:USB_Micro-B_Molex_47346-0001, symbol Connector:USB_B_Micro
- added J3: plate, lightring:touchplate, symbol Connector:Conn_01x01_Female
- added R45: 12k, Resistor_SMD:R_0603_1608Metric, symbol Device:R
- added R46: 100k, Resistor_SMD:R_0603_1608Metric, symbol Device:R
- added R47: 1M, Resistor_SMD:R_0603_1608Metric, symbol Device:R
- added R48: 470R, Resistor_SMD:R_0603_1608Metric, symbol Device:R
- added R49: 10k, Resistor_SMD:R_0603_1608Metric, symbol Device:R
- added U2: MCP73831-2-OT, Package_TO_SOT_SMD:SOT-23-5, symbol Battery_Management:MCP73831-2-OT
- added U3: AT42QT1012-T, Package_TO_SOT_SMD:SOT-23-6, symbol Sensor_Touch:AT42QT1012-T
- added U4: LDK130-33_SOT23_SOT353, Package_TO_SOT_SMD:SOT-23-5, symbol Regulator_Linear:LDK130-33_SOT23_SOT353
- BT1: footprint Battery:BatteryHolder_Keystone_500 -> Resistor_SMD:R_1206_3216Metric
- C1, C2, C4, C5, C6, C7, C8: footprint lightring:LC_CAP -> Capacitor_SMD:C_0603_1608Metric
- R43, R44: footprint lightring:LR_RES -> Resistor_SMD:R_0603_1608Metric
Connections:
- net GND: now also C10.2, C12.2, C9.2, J2.5 (GND), R45.2, R46.2, R47.2, U2.2 (VSS), U3.2 (VSS), U3.6 (TIME), U4.2 (GND)
- net VCC: now also C12.1, U2.3 (VBAT), U4.1 (IN), U4.3 (EN); no longer C2.1, C6.1, C7.1, C8.1, R43.1, U1.6 (Vbat), U1.7 (Vref), U1.8 (Vdd)
- net TOUCH: now reaches U1.14 (PC1)
- net TOUCH: now also R46.1, U3.1 (OUT)
- new net: R48.1, U2.1 (STAT)
- new net: R45.1, U2.5 (PROG)
- new net: D44.1 (K), R48.2
- new net: C11.1, R49.2, U3.3 (SNSK)
- new net: C11.2, R47.1, U3.4 (SNS)
- new net: J3.1 (Pin_1), R49.1
- new net +3V3: C10.1, C2.1, C6.1, C7.1, C8.1, R43.1, U1.6 (Vbat), U1.7 (Vref), U1.8 (Vdd), U3.5 (VDD), U4.5 (OUT)
- new net +5V: C9.1, D44.2 (A), J2.1 (VBUS), U2.4 (VDD)
- no-connect marks 11 -> 14
Other:
- moved on the sheet: BT1, C1, C2, C4, C5, C6, C7, C8, D16, D17, D18, D19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

Commit message: testing program
Connections:
- net WAKE: no longer names the net of U1.41 (PD9)
Changed lines of the file:
@@
 Text GLabel 9500 3600 0    50   Input ~ 0
 M23
-Text GLabel 9500 4900 0    50   Input ~ 0
-WAKE
 Text GLabel 9500 5000 0    50   Input ~ 0
 M5

Commit message: initial program
Connections:
- net XTAL1: now also U1.4 (PC14); no longer U1.3 (PC13)
- net XTAL2: now also U1.5 (PC15); no longer U1.4 (PC14)
- no-connect marks 14 -> 15
Changed lines of the file:
@@
 Wire Wire Line
 	9200 2700 9500 2700
-Text GLabel 9500 2800 0    50   Input ~ 0
+Text GLabel 9500 2900 0    50   Input ~ 0
 XTAL1
-Text GLabel 9500 2900 0    50   Input ~ 0
+Text GLabel 9500 3000 0    50   Input ~ 0
 XTAL2
 Text GLabel 9500 5100 0    50   Input ~ 0
@@
 WORK
 NoConn ~ 9500 4700
+NoConn ~ 9500 3300
 NoConn ~ 9500 3200
-NoConn ~ 9500 3100
 $Comp
 L Device:R R44
@@
 Text GLabel 9500 4600 0    50   Input ~ 0
 TOUCH
+NoConn ~ 9500 2800
 $EndSCHEMATC

Commit message: working program
Parts:
- J2: symbol Connector:USB_B_Micro -> lightring-rescue:USB_B_Micro-Connector
Changed lines of the file:
@@
 EESchema Schematic File Version 4
+LIBS:lightring-cache
 EELAYER 30 0
 EELAYER END
@@
 Connection ~ 8400 1500
 $Comp
-L Connector:USB_B_Micro J2
+L lightring-rescue:USB_B_Micro-Connector J2
 U 1 1 5FF3E4D7
 P 4450 1100

Commit message: v0.3 PCB
Parts:
- added C3: 104, Capacitor_SMD:C_0603_1608Metric, symbol Device:C
- added R50, R51: 100k, Resistor_SMD:R_0603_1608Metric, symbol Device:R
- BT1: footprint Resistor_SMD:R_1206_3216Metric -> Resistor_SMD:R_1210_3225Metric
Connections:
- net GND: now also C3.2, R51.2
- net M20: now also U1.41 (PD9); no longer U1.17 (PA0)
- net VCC: now also R50.1
- new net STATE: C3.1, R50.2, R51.1, U1.17 (PA0)
- no-connect marks 15 -> 14
Changed lines of the file:
@@
 EESchema Schematic File Version 4
-LIBS:lightring-cache
 EELAYER 30 0
 EELAYER END
@@
 Text GLabel 9500 5600 0    50   Input ~ 0
 M29
-Text GLabel 10500 2750 2    50   Input ~ 0
+Text GLabel 9500 4900 0    50   Input ~ 0
 M20
 Text GLabel 10500 2850 2    50   Input ~ 0
@@
 F 0 "BT1" H 7268 1146 50  0000 L CNN
 F 1 "Battery_Cell" H 7268 1055 50  0000 L CNN
-F 2 "Resistor_SMD:R_1206_3216Metric" V 7150 1110 50  0001 C CNN
+F 2 "Resistor_SMD:R_1210_3225Metric" V 7150 1110 50  0001 C CNN
 F 3 "~" V 7150 1110 50  0001 C CNN
 	1    7150 1050
@@
 Text GLabel 8250 5700 0    50   Input ~ 0
 SET
-NoConn ~ 7800 5400
 Text GLabel 9500 4600 0    50   Input ~ 0
 TOUCH
 NoConn ~ 9500 2800
+$Comp
+L Device:R R50
+U 1 1 600E0A15
+P 6150 5300
+F 0 "R50" H 6220 5346 50  0000 L CNN
+F 1 "100k" H 6220 5255 50  0000 L CNN
+F 2 "Resistor_SMD:R_0603_1608Metric" V 6080 5300 50  0001 C CNN
+F 3 "~" H 6150 5300 50  0001 C CNN
+	1    6150 5300
+	1    0    0    -1
+$EndComp
+$Comp
+L Device:R R51
+U 1 1 600E16F0
+P 6150 5700
+F 0 "R51" H 6220 5746 50  0000 L CNN
+F 1 "100k" H 6220 5655 50  0000 L CNN
+F 2 "Resistor_SMD:R_0603_1608Metric" V 6080 5700 50  0001 C CNN
+F 3 "~" H 6150 5700 50  0001 C CNN
+	1    6150 5700
+	1    0    0    -1
+$EndComp
+$Comp
+L power:GND #PWR0113
+U 1 1 600E3242
+P 6150 5950
+F 0 "#PWR0113" H 6150 5700 50  0001 C CNN
+F 1 "GND" H 6155 5777 50  0000 C CNN
+F 2 "" H 6150 5950 50  0001 C CNN
+F 3 "" H 6150 5950 50  0001 C CNN
+	1    6150 5950
+	1    0    0    -1
+$EndComp
+$Comp
+L power:VCC #PWR0114
+U 1 1 600EB1AD
+P 6150 5100
+F 0 "#PWR0114" H 6150 4950 50  0001 C CNN
+F 1 "VCC" H 6165 5273 50  0000 C CNN
+F 2 "" H 6150 5100 50  0001 C CNN
+F 3 "" H 6150 5100 50  0001 C CNN
+	1    6150 5100
+	1    0    0    -1
+$EndComp
+Wire Wire Line
+	6150 5100 6150 5150
+Wire Wire Line
+	6150 5950 6150 5850
+Wire Wire Line
+	6150 5550 6150 5450
+$Comp
+L Device:C C3
+U 1 1 6010184D
+P 6600 5700
+F 0 "C3" H 6715 5746 50  0000 L CNN
+F 1 "104" H 6715 5655 50  0000 L CNN
+F 2 "Capacitor_SMD:C_0603_1608Metric" H 6638 5550 50  0001 C CNN
+F 3 "~" H 6600 5700 50  0001 C CNN
+	1    6600 5700
+	1    0    0    -1
+$EndComp
+Wire Wire Line
+	6150 5550 6600 5550
+Connection ~ 6150 5550
+Wire Wire Line
+	6150 5850 6600 5850
+Connection ~ 6150 5850
+Text GLabel 6950 5550 2    50   Input ~ 0
+STATE
+Wire Wire Line
+	6600 5550 6950 5550
+Connection ~ 6600 5550
+Text GLabel 10500 2750 2    50   Input ~ 0
+STATE
 $EndSCHEMATC

Commit message: changed stabiliser
Parts:
- U4: value LDK130-33_SOT23_SOT353 -> TC1185-3.3
Changed lines of the file:
@@
 P 8400 950
 F 0 "U4" H 8400 1292 50  0000 C CNN
-F 1 "LDK130-33_SOT23_SOT353" H 8400 1201 50  0000 C CNN
+F 1 "TC1185-3.3" H 8400 1201 50  0000 C CNN
 F 2 "Package_TO_SOT_SMD:SOT-23-5" H 8400 1275 50  0001 C CNN
 F 3 "http://www.st.com/content/ccc/resource/technical/document/datasheet/29/10/f7/87/2f/66/47/f4/DM00076097.pdf/files/DM00076097.pdf/jcr:content/translations/en.DM00076097.pdf" H 8400 950 50  0001 C CNN
