File: doc/case/base/base.kicad_pcb (KiCad board)
At the start: 2 copper layers, 44 x 56 mm, 0 parts

Commit message: v2 base board
Other:
- board size 44 x 56 mm -> 44 x 51 mm
Changed lines of the file:
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@@
       (outputformat 1)
       (mirror false)
-      (drillshape 1)
+      (drillshape 0)
       (scaleselection 1)
-      (outputdirectory ""))
+      (outputdirectory "output/V2/"))
   )
   (net 0 "")
@@
   (gr_arc (start 130 90) (end 144.199999 106.799999) (angle -99.58846413) (layer Edge.Cuts) (width 0.05))
   (gr_arc (start 130 90) (end 115.800001 73.200001) (angle -99.58846413) (layer Edge.Cuts) (width 0.05))
-  (gr_line (start 142.1 116) (end 117.9 116) (layer Edge.Cuts) (width 0.05))
-  (gr_line (start 117.9 114) (end 142.1 114) (layer Edge.Cuts) (width 0.05))
-  (gr_line (start 117.9 116) (end 117.9 114) (layer Edge.Cuts) (width 0.05))
-  (gr_line (start 142.1 114) (end 142.1 116) (layer Edge.Cuts) (width 0.05))
-  (gr_line (start 144.2 106.8) (end 144.2 118) (layer Edge.Cuts) (width 0.05))
-  (gr_line (start 115.8 106.8) (end 115.8 118) (layer Edge.Cuts) (width 0.05))
-  (gr_line (start 144.2 118) (end 115.8 118) (layer Edge.Cuts) (width 0.05))
-  (gr_line (start 117.9 66) (end 117.9 64) (layer Edge.Cuts) (width 0.05))
-  (gr_line (start 142.1 66) (end 117.9 66) (layer Edge.Cuts) (width 0.05))
-  (gr_line (start 142.1 64) (end 142.1 66) (layer Edge.Cuts) (width 0.05))
-  (gr_line (start 117.9 64) (end 142.1 64) (layer Edge.Cuts) (width 0.05))
-  (gr_line (start 144.2 73.2) (end 144.2 62) (layer Edge.Cuts) (width 0.05))
+  (gr_line (start 142.1 113.5) (end 117.9 113.5) (layer Edge.Cuts) (width 0.05))
+  (gr_line (start 117.9 111.5) (end 142.1 111.5) (layer Edge.Cuts) (width 0.05))
+  (gr_line (start 117.9 113.5) (end 117.9 111.5) (layer Edge.Cuts) (width 0.05))
+  (gr_line (start 142.1 111.5) (end 142.1 113.5) (layer Edge.Cuts) (width 0.05))
+  (gr_line (start 144.2 106.8) (end 144.2 115.5) (layer Edge.Cuts) (width 0.05))
+  (gr_line (start 115.8 106.8) (end 115.8 115.5) (layer Edge.Cuts) (width 0.05))
+  (gr_line (start 144.2 115.5) (end 115.8 115.5) (layer Edge.Cuts) (width 0.05))
+  (gr_line (start 117.9 68.5) (end 117.9 66.5) (layer Edge.Cuts) (width 0.05))
+  (gr_line (start 142.1 68.5) (end 117.9 68.5) (layer Edge.Cuts) (width 0.05))
+  (gr_line (start 142.1 66.5) (end 142.1 68.5) (layer Edge.Cuts) (width 0.05))
+  (gr_line (start 117.9 66.5) (end 142.1 66.5) (layer Edge.Cuts) (width 0.05))
+  (gr_line (start 144.2 73.2) (end 144.2 64.5) (layer Edge.Cuts) (width 0.05))
   (gr_line (start 142 73.6) (end 144.2 73.6) (layer Eco1.User) (width 0.1))
-  (gr_line (start 115.8 62) (end 144.2 62) (layer Edge.Cuts) (width 0.05))
-  (gr_line (start 115.8 73.2) (end 115.8 62) (layer Edge.Cuts) (width 0.05))
+  (gr_line (start 115.8 64.5) (end 144.2 64.5) (layer Edge.Cuts) (width 0.05))
+  (gr_line (start 115.8 73.2) (end 115.8 64.5) (layer Edge.Cuts) (width 0.05))
   (gr_line (start 142.9 85.3) (end 146.7 85.3) (layer Eco1.User) (width 0.15))
   (gr_circle (center 144.8 85.3) (end 146.7 85.3) (layer Eco2.User) (width 0.15))

Commit message: changed to mk2 in base
Other:
- board text added: "lightring Mk2"
- board text removed: "lightring Mk1"
Changed lines of the file:
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@@
     (effects (font (size 1 1) (thickness 0.15)) (justify mirror))
   )
-  (gr_text "lightring Mk1" (at 129.9 90.4) (layer B.SilkS)
+  (gr_text "lightring Mk2" (at 129.9 90.4) (layer B.SilkS)
     (effects (font (size 3 3) (thickness 0.5)) (justify mirror))
   )
